Commit message: finished initial bot description

File: src/robot_description/description/robot_core.xacro (robot description, xacro)
@@ -2,4 +2,6 @@
 <!-- Following: https://www.youtube.com/watch?v=BcjHyhV0kIs -->
 <robot xmlns:xacro="http://www.ros.org/wiki/xacro" >
+    <!-- Import intertia macros so they're easier to define-->
+    <xacro:include filename="intertial_macros.xacro" />
     <material name="white">
         <color rgba="1 1 1 1" />
@@ -14,6 +16,8 @@
         <color rgba="0 0 0 1" />
     </material>
+    <!-- Base Link -->
     <link name="base_link">
     </link>
+    <!-- Chassis Link -->
     <joint name="chassis_joint" type="fixed">
         <parent link="base_link" />
@@ -29,4 +33,85 @@
             <material name="white" />
         </visual>
+        <collision>
+            <origin xyz="0.15 0 0.075" />
+            <geometry>
+                <box size="0.3 0.3 0.15" />
+            </geometry>
+        </collision>
+        <xacro:inertial_box mass="0.5" x="0.3" y="0.3" z="0.15">
+            <origin xyz="0.15 0 0.075"  rpy="0 0 0 "/>
+        </xacro:inertial_box>
+    </link>
+    <!-- Left Wheel Link -->
+    <joint name="left_wheel_joint" type="continuous">
+        <parent link="base_link" />
+        <child link="left_wheel" />
+        <!-- cylinders are oriented in z axis by default so we need to rotate  along x axis (right hand rule for sign)-->
+        <origin xyz="0 0.175 0" rpy="-${pi/2} 0 0" />
+        <!-- define the positve forward motion; since we rotated the wheel, the z axis is now pointing where y was so we want to rotate around z-->
+        <axis xyz="0 0 1" />
+    </joint>
+    <link name="left_wheel">
+        <visual>
+            <geometry>
+                <cylinder radius="0.05" length="0.04" /> <!-- 50 mm and 40 mm-->
+            </geometry>
+            <material name="blue" />
+        </visual>
+        <collision>
+            <geometry>
+                <cylinder radius="0.05" length="0.04" /> <!-- 50 mm and 40 mm-->
+            </geometry>
+        </collision>
+        <xacro:inertial_cylinder mass="0.1" length="0.04" radius="0.05">
+            <origin xyz="0 0 0"  rpy="0 0 0"/>
+        </xacro:inertial_cylinder>
+    </link>
+    <!-- Right Wheel Link -->
+    <joint name="right_wheel_joint" type="continuous">
+        <parent link="base_link" />
+        <child link="right_wheel" />
+        <!-- cylinders are oriented in z axis by default so we need to rotate  along x axis (right hand rule for sign)-->
+        <origin xyz="0 -0.175 0" rpy="${pi/2} 0 0" />
+        <!-- define the positve forward motion; since we rotated the wheel, the z axis is now pointing where y was so we want to rotate around z-->
+        <axis xyz="0 0 -1" />
+    </joint>
+    <link name="right_wheel">
+        <visual>
+            <geometry>
+                <cylinder radius="0.05" length="0.04" /> <!-- 50 mm and 40 mm-->
+            </geometry>
+            <material name="blue" />
+        </visual>
+        <collision>
+            <geometry>
+                <cylinder radius="0.05" length="0.04" /> <!-- 50 mm and 40 mm-->
+            </geometry>
+        </collision>
+        <xacro:inertial_cylinder mass="0.1" length="0.04" radius="0.05">
+            <origin xyz="0 0 0"  rpy="0 0 0"/>
+        </xacro:inertial_cylinder>
+    </link>
+    <!-- Caster Wheel Link -->
+    <joint name="caster_wheel_joint" type="fixed">
+        <parent link="chassis" />
+        <child link="caster_wheel" />
+        <origin xyz="0.24 0 0"/> <!-- Close to the front of the bot -->
+    </joint>
+    <link name="caster_wheel">
+        <visual>
+            <geometry>
+                <sphere radius="0.05" />
+            </geometry>
+            <material name="black" />
+        </visual>
+        <collision>
+            <geometry>
+                <sphere radius="0.05" />
+            </geometry>
+        </collision>
+        <xacro:inertial_sphere mass="0.1" radius="0.05">
+            <origin xyz="0 0 0" rpy="0 0 0 " />
+        </xacro:inertial_sphere>
     </link>
 </robot>
