Commit message: fixed the robot driving

File: src/robot_description/description/robot.urdf.xacro (robot description, xacro)
@@ -1,4 +1,6 @@
 <?xml version="1.0"?>
 <robot xmlns:xacro="http://www.ros.org/wiki/xacro" name="robot">
+    <!-- Robot description-->
     <xacro:include filename="robot_core.xacro" />
+    <xacro:include filename="gazebo_control.xacro" />
 </robot>

File: src/robot_description/description/robot_core.xacro (robot description, xacro)
@@ -4,6 +4,6 @@
     <!-- Import intertia macros so they're easier to define-->
     <xacro:include filename="intertial_macros.xacro" />
-    <material name="white">
-        <color rgba="1 1 1 1" />
+    <material name="off_white">
+        <color rgba="0.9 0.9 0.9 1" />
     </material>
     <material name="orange">
@@ -31,5 +31,5 @@
                 <box size="0.3 0.3 0.15" />
             </geometry>
-            <material name="white" />
+            <material name="off_white" />
         </visual>
         <collision>
